File: electronics/pingpong-scoreboard/pingpong-scoreboard.kicad_pcb (KiCad board)
At the start: 2 copper layers, 116.8 x 57.2 mm, 27 parts, among them J1 Conn_01x02_Male, J2 Conn_01x02_Male, J3 Conn_01x02_Male, J4 Conn_02x03_Odd_Even, J5 USB_B_Micro, SW1 SW_DPDT_x2, SW2 SW_DPDT_x2, SW3 SW_DPDT_x2, U1 ATtiny84-20PU, U2 MAX7219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

Commit message: Route PCB, set up nice silkscreen
Parts:
- added G***: LOGO, m-logo:m-logo, F.Cu at (194.3, 95.5)
- moved C5 2.54 mm to (144.8, 118.1), turned to 0 degrees
Routing:
- net /DIG4: track 0.00 -> 210.7 mm, vias 0 -> 1
- net /SEG_A: track 0.00 -> 154.7 mm
- net +5V: track 0.00 -> 123.0 mm
- net /SEG_B: track 0.00 -> 111.0 mm, vias 0 -> 4
- net /PA5: track 0.00 -> 98.9 mm
- net /DIG2: track 0.00 -> 90.3 mm, vias 0 -> 2
- net /DIG1: track 0.00 -> 83.8 mm, vias 0 -> 2
- net /PA2: track 0.00 -> 83.5 mm
- net /DIG5: track 0.00 -> 70.1 mm
- net /PA4: track 0.00 -> 68.0 mm, vias 0 -> 2
- net /SEG_F: track 0.00 -> 67.4 mm
- net /PA7: track 0.00 -> 65.3 mm, vias 0 -> 3
- net /PA6: track 0.00 -> 56.4 mm, vias 0 -> 2
- net /DIG0: track 0.00 -> 55.8 mm, vias 0 -> 1
- net /SEG_C: track 0.00 -> 48.5 mm
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- added copper zone on B.Cu, net GND
- added copper zone on F.Cu, net GND
Other:
- board size 116.8 x 57.2 mm -> 116.8 x 58.4 mm
- net class Power added: clearance 0.2, trace_width 0.4, via_dia 0.8, via_drill 0.4
- board text added: "+"
- board text added: "ALL-TIME"
- board text added: "AVR ISP"
- board text added: "DISPLAY/LEDS DRIVER"
- board text added: "GAME"
- board text added: "JLCJLCJLCJLC"
- board text added: "MFR. Order No.:"
- board text added: "MICHD - NOV 2019"
- board text added: "MICRO USB (POWER)"
- board text added: "MICROCONTROLLER"
- board text added: "MICROCONTROLLER PROGRAMMING CONNECTOR"
- board text added: "MODE"
- board text added: "PIEZO SPEAKER"
- board text added: "PING-PONG SCOREBOARD REV.0"
- board text added: "PLAYER 1"
- board text added: "PLAYER 1 EXT. BUTTON"
- board text added: "PLAYER 2"
- board text added: "PLAYER 2 EXT. BUTTON"
- board text added: "SET"
