File: electronics/pingpong-scoreboard/pingpong-scoreboard.sch (KiCad schematic (older format))
At the start: 24 parts, among them J1 Conn_01x02_Male, J2 Conn_01x02_Male, J3 Conn_02x03_Odd_Even, J4 USB_B_Micro, SW1 SW_DPDT_x2, SW2 SW_DPDT_x2, SW3 SW_DPDT_x2, U1 ATtiny84-20PU, U2 MAX7219, U3 TOF-5461AG-1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

Commit message: Lay out PCB components + add piezo output
Parts:
- added C6: 330n, Capacitor_SMD:C_0603_1608Metric, symbol Device:C
- added J3: Conn_01x02_Male, Connector_PinHeader_2.54mm:PinHeader_1x02_P2.54mm_Horizontal, symbol Connector:Conn_01x02_Male
- added R3: 1k, Resistor_SMD:R_0603_1608Metric, symbol Device:R
- C1, C2, C3, C4: footprint (none) -> Capacitor_THT:C_Disc_D4.3mm_W1.9mm_P5.00mm
- C5: footprint (none) -> Capacitor_THT:CP_Radial_D6.3mm_P2.50mm
- D1, D2: footprint (none) -> LED_THT:LED_D5.0mm_Clear
- D3, D4, D5: footprint (none) -> LED_THT:LED_D5.0mm
- D6: footprint (none) -> LED_SMD:LED_0603_1608Metric
- J1, J2: footprint (none) -> Connector_PinHeader_2.54mm:PinHeader_1x02_P2.54mm_Horizontal
- J4: renamed from J3; footprint (none) -> Connector_IDC:IDC-Header_2x03_P2.54mm_Horizontal
- J5: renamed from J4; footprint (none) -> Connector_USB:USB_Micro-B_Amphenol_10103594-0001LF_Horizontal
- R1, R2: footprint (none) -> Resistor_SMD:R_0603_1608Metric
- SW1, SW2, SW3: footprint (none) -> 6-pin-momentary-push-button:6-pin-momentary-push-button
- U1: footprint Package_DIP:DIP-14_W7.62mm -> Package_DIP:DIP-14_W7.62mm_LongPads
- U2: footprint (none) -> Package_DIP:DIP-24_W7.62mm_LongPads
- Y1: footprint (none) -> Crystal:Resonator-2Pin_W10.0mm_H5.0mm
Connections:
- net GND: now also J3.2 (Pin_2)
- net PA6: now also R3.2
- new net: C6.2, R3.1
- new net PIEZO: C6.1, J3.1 (Pin_1)
Other:
- moved on the sheet: J1, J2, J5
